Commit message: feat(robotiq_description): run the real driver asynchronously in ros2_control
New arguments scheduling_policy, rw_rate, thread_priority and cpu_affinity,
through robotiq_control.launch.py and the xacro chain of both 2F models. They
set the <ros2_control> tag's is_async and rw_rate and its <properties><async>,
as the UR and Franka descriptions do. An empty scheduling_policy (default)
keeps the driver synchronous; mock hardware and the simulator plugins always
stay synchronous.

The launch file's hardware_component_names() now finds the component name in
any attribute order: xacro writes attributes alphabetically, so is_async now
comes before name.

Co-Authored-By: Carl <carl@b-robotized.ai>

File: grippers/robotiq_description/urdf/2f_140.ros2_control.xacro (robot description, xacro)
@@ -16,4 +16,8 @@
         tcp_host:=''
         tcp_port:=54321
+        rw_rate:=0
+        scheduling_policy:=''
+        thread_priority:=50
+        cpu_affinity:=''
         gripper_speed_multiplier:=1.0
         gripper_force_multiplier:=0.5
@@ -21,5 +25,13 @@
         gripper_max_force:=125.0
         gripper_closed_position:=0.695">
-        <ros2_control name="${name}" type="system">
+        <!-- Async only for the real driver: the mock and simulator plugins stay in the
+             controller manager's loop. An empty scheduling_policy keeps it synchronous. -->
+        <xacro:property name="is_async" value="${scheduling_policy != '' and not (use_fake_hardware or sim_gazebo or sim_topic_based)}"/>
+        <ros2_control name="${name}" type="system" rw_rate="${rw_rate}" is_async="${is_async}">
+            <xacro:robotiq_2f_async_properties
+                is_async="${is_async}"
+                scheduling_policy="${scheduling_policy}"
+                thread_priority="${thread_priority}"
+                cpu_affinity="${cpu_affinity}"/>
             <!-- Plugins -->
             <xacro:robotiq_2f_hardware

File: grippers/robotiq_description/urdf/2f_85.ros2_control.xacro (robot description, xacro)
@@ -16,4 +16,8 @@
         tcp_host:=''
         tcp_port:=54321
+        rw_rate:=0
+        scheduling_policy:=''
+        thread_priority:=50
+        cpu_affinity:=''
         gripper_speed_multiplier:=1.0
         gripper_force_multiplier:=0.5
@@ -21,5 +25,13 @@
         gripper_max_force:=235.0
         gripper_closed_position:=0.7929">
-        <ros2_control name="${name}" type="system">
+        <!-- Async only for the real driver: the mock and simulator plugins stay in the
+             controller manager's loop. An empty scheduling_policy keeps it synchronous. -->
+        <xacro:property name="is_async" value="${scheduling_policy != '' and not (use_fake_hardware or sim_gazebo or sim_topic_based)}"/>
+        <ros2_control name="${name}" type="system" rw_rate="${rw_rate}" is_async="${is_async}">
+            <xacro:robotiq_2f_async_properties
+                is_async="${is_async}"
+                scheduling_policy="${scheduling_policy}"
+                thread_priority="${thread_priority}"
+                cpu_affinity="${cpu_affinity}"/>
             <!-- Plugins -->
             <xacro:robotiq_2f_hardware

File: grippers/robotiq_description/urdf/2f_common.ros2_control.xacro (robot description, xacro)
@@ -53,4 +53,18 @@
         </hardware>
     </xacro:macro>
+    <!-- The <properties> of an async component. rw_rate and is_async are attributes of
+         the <ros2_control> tag itself, set by the model's ros2_control xacro. -->
+    <xacro:macro name="robotiq_2f_async_properties" params="is_async scheduling_policy thread_priority cpu_affinity">
+        <xacro:if value="${is_async}">
+            <properties>
+                <xacro:if value="${cpu_affinity == ''}">
+                    <async scheduling_policy="${scheduling_policy}" thread_priority="${thread_priority}" print_warnings="true"/>
+                </xacro:if>
+                <xacro:unless value="${cpu_affinity == ''}">
+                    <async scheduling_policy="${scheduling_policy}" thread_priority="${thread_priority}" affinity="${cpu_affinity}" print_warnings="true"/>
+                </xacro:unless>
+            </properties>
+        </xacro:if>
+    </xacro:macro>
     <!-- A mimic joint the simulator owns: declared so /joint_states carries it,
          but never commanded. Gazebo derives mimic joints itself, so it gets no

File: grippers/robotiq_description/urdf/robotiq_2f_140_macro.urdf.xacro (robot description, xacro)
@@ -21,4 +21,8 @@
         tcp_host:=''
         tcp_port:=54321
+        rw_rate:=0
+        scheduling_policy:=''
+        thread_priority:=50
+        cpu_affinity:=''
         gripper_speed_multiplier:=1.0
         gripper_force_multiplier:=0.5
@@ -52,4 +56,8 @@
                 tcp_host="${tcp_host}"
                 tcp_port="${tcp_port}"
+                rw_rate="${rw_rate}"
+                scheduling_policy="${scheduling_policy}"
+                thread_priority="${thread_priority}"
+                cpu_affinity="${cpu_affinity}"
                 gripper_speed_multiplier="${gripper_speed_multiplier}"
                 gripper_force_multiplier="${gripper_force_multiplier}"

File: grippers/robotiq_description/urdf/robotiq_2f_85_macro.urdf.xacro (robot description, xacro)
@@ -21,4 +21,8 @@
         tcp_host:=''
         tcp_port:=54321
+        rw_rate:=0
+        scheduling_policy:=''
+        thread_priority:=50
+        cpu_affinity:=''
         gripper_speed_multiplier:=1.0
         gripper_force_multiplier:=0.5
@@ -52,4 +56,8 @@
                 tcp_host="${tcp_host}"
                 tcp_port="${tcp_port}"
+                rw_rate="${rw_rate}"
+                scheduling_policy="${scheduling_policy}"
+                thread_priority="${thread_priority}"
+                cpu_affinity="${cpu_affinity}"
                 gripper_speed_multiplier="${gripper_speed_multiplier}"
                 gripper_force_multiplier="${gripper_force_multiplier}"

File: grippers/robotiq_description/urdf/robotiq_2f_gripper.urdf.xacro (robot description, xacro)
@@ -12,4 +12,9 @@
     <xacro:arg name="tcp_host" default="" />
     <xacro:arg name="tcp_port" default="54321" />
+    <!-- ros2_control async execution; an empty scheduling_policy keeps the driver synchronous. -->
+    <xacro:arg name="rw_rate" default="0" />
+    <xacro:arg name="scheduling_policy" default="" />
+    <xacro:arg name="thread_priority" default="50" />
+    <xacro:arg name="cpu_affinity" default="" />
     <xacro:arg name="sim_topic_based" default="false" />
     <xacro:arg name="sim_joint_commands_topic" default="/sim/joint_commands" />
@@ -24,4 +29,6 @@
     <xacro:robotiq_gripper name="RobotiqGripperHardwareInterface" prefix="" parent="world" use_fake_hardware="$(arg use_fake_hardware)" com_port="$(arg com_port)" baudrate="$(arg baudrate)"
         transport="$(arg transport)" tcp_host="$(arg tcp_host)" tcp_port="$(arg tcp_port)"
+        rw_rate="$(arg rw_rate)" scheduling_policy="$(arg scheduling_policy)"
+        thread_priority="$(arg thread_priority)" cpu_affinity="$(arg cpu_affinity)"
         sim_topic_based="$(arg sim_topic_based)"
         sim_joint_commands_topic="$(arg sim_joint_commands_topic)" sim_joint_states_topic="$(arg sim_joint_states_topic)"
